File: AMP.kicad_sch (KiCad schematic)
At the start: 62 parts, among them Q1 IRF9610PBF, Q11 BCP56-16,115, Q12 BCP56-16,115, Q2 IRF9610PBF, Q3 IRF9610PBF, Q4 IRFP240PBF, Q5 IRFP240PBF, Q6 IRFP240PBF, Q7 IRFP240PBF, Q8 IRFP240PBF, Q9 IRFP240PBF

Commit message: fix some bugs
Parts:
- Q1, Q2, Q3: footprint 3rd package:IRF9610PBF -> cus_mosfet:IRF9610PBF
- Q4, Q5, Q6, Q7, Q8, Q9: footprint 3rd package:IRFP240PBF -> cus_mosfet:IRFP240PBF
Changed lines of the file:
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@@
 			)
 		)
-		(property "Footprint" "3rd package:IRFP240PBF"
+		(property "Footprint" "cus_mosfet:IRFP240PBF"
 			(at 208.28 48.26 0)
 			(effects
@@
 			)
 		)
-		(property "Footprint" "3rd package:IRF9610PBF"
+		(property "Footprint" "cus_mosfet:IRF9610PBF"
 			(at 68.58 46.99 0)
 			(effects
@@
 			)
 		)
-		(property "Footprint" "3rd package:IRFP240PBF"
+		(property "Footprint" "cus_mosfet:IRFP240PBF"
 			(at 208.28 130.81 0)
 			(effects
@@
 			)
 		)
-		(property "Footprint" "3rd package:IRF9610PBF"
+		(property "Footprint" "cus_mosfet:IRF9610PBF"
 			(at 66.04 86.36 0)
 			(effects
@@
 			)
 		)
-		(property "Footprint" "3rd package:IRFP240PBF"
+		(property "Footprint" "cus_mosfet:IRFP240PBF"
 			(at 180.34 48.26 0)
 			(effects
@@
 			)
 		)
-		(property "Footprint" "3rd package:IRFP240PBF"
+		(property "Footprint" "cus_mosfet:IRFP240PBF"
 			(at 231.14 130.81 0)
 			(effects
@@
 			)
 		)
-		(property "Footprint" "3rd package:IRFP240PBF"
+		(property "Footprint" "cus_mosfet:IRFP240PBF"
 			(at 231.14 48.26 0)
 			(effects
@@
 			)
 		)
-		(property "Footprint" "3rd package:IRFP240PBF"
+		(property "Footprint" "cus_mosfet:IRFP240PBF"
 			(at 180.34 130.81 0)
 			(effects
@@
 			)
 		)
-		(property "Footprint" "3rd package:IRF9610PBF"
+		(property "Footprint" "cus_mosfet:IRF9610PBF"
 			(at 82.55 86.36 0)
 			(effects
