File: PASS A5功放.kicad_pcb (KiCad board)
At the start: 6 copper layers, 200 x 100 mm, 109 parts, among them IC1 OPA1611AIDR, IC2 LM317AEMPX_NOPB, IC3 LM337IMP_NOPB, Q1 IRF9610PBF, Q11 BCP56-16,115, Q12 BCP56-16,115, Q2 IRF9610PBF, Q3 IRF9610PBF, Q4 IRFP240PBF, Q5 IRFP240PBF, Q6 IRFP240PBF, Q7 IRFP240PBF, Q8 IRFP240PBF, Q9 IRFP240PBF, U1 UPC1237HA, U2 SFH6206-2T

Commit message: fix some bugs
Parts:
- moved C26 0.40 mm to (274.9, 132.1)
- moved C13 0.40 mm to (284.0, 135.9)
- moved C14 0.40 mm to (245.5, 140.9)
- moved C25 0.05 mm to (258.9, 132.1)
Routing:
- net /VIN: track 208.3 -> 219.1 mm, vias 5 -> 3
- net /UPC1237_PIN4: track 57.2 -> 46.5 mm, vias 1 -> 3
- net /DC 35V: track 108.8 -> 106.3 mm, vias 4 -> 5
- net Net-(D4-A): track 73.9 -> 72.5 mm, vias 0 -> 2
- net Net-(D3-K): track 69.6 -> 71.0 mm
- net /UPC1237_PIN8: track 42.2 -> 41.1 mm
- net Net-(IC1-+IN): track 33.2 -> 32.4 mm
